Commit message: add files force to torque

File: julia/odes/pendu.urdf (robot description, URDF)
Before this commit: robot DoublePendulum, 3 links, 2 joints
Links:
- added link endeffector, mass 0; visual box size=0.05 0.05 0.05
- link base_link: geometry 
- link lower_link: geometry visual cylinder length=2 radius=.05
- link upper_link: geometry visual box size=0.05 0.05 1.0
Joints:
- added joint endjoint: type fixed, parent lower_link, child endeffector, origin xyz=0.0 0.0 -2 rpy=0.0 0 0 
- joint shoulder: axis 0 0 1 -> 0 1 0
