Commit message: changes to planar3R code

File: julia/odes/planar3R.urdf (robot description, URDF)
Before this commit: robot ThreeLinkPlanar, 5 links, 4 joints
Links:
- removed link lower_link
- removed link lowest_link
- removed link upper_link
- added link blue_link, mass 1; visual box size=1.0 0.05 0.05
- added link green_link, mass 1; visual box size=1.05 0.05 0.05
- added link red_link, mass 1; visual box size=1.0 0.05 0.05
Joints:
- joint elbow: axis 0 0 1 -> 0 1 0; child lower_link -> blue_link; parent upper_link -> red_link
- joint endjoint: origin xyz=1.0 0.0 0 rpy=0.0 0 0  -> xyz=1.0 0.0 0 rpy=0.0 0 0.0 ; parent lowest_link -> green_link
- joint shoulder: child upper_link -> red_link
- joint wrist: child lowest_link -> green_link; parent lower_link -> blue_link
